File: NEW.kicad_pcb (KiCad board)
At the start: 2 copper layers, 135.3 x 80 mm, 21 parts, among them J1 Screw_Terminal_01x16, J2 Screw_Terminal_01x16, J3 buck converter, J4 Infrared, J5 BMI, J6 light sensor, J7 servo, J8 Screw_Terminal_01x03, J9 battery +, Q1 PN2222A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

Commit message: 2.0
Parts:
- added C4: C_Polarized_Small, Capacitor_THT:C_Disc_D3.8mm_W2.6mm_P2.50mm, F.Cu at (105.2, 59.8)
- added J10: boost conv (IN), TerminalBlock:TerminalBlock_Altech_AK300-2_P5.00mm, F.Cu at (92.8, 101.0)
- added J11: Battery, TerminalBlock:TerminalBlock_Altech_AK300-2_P5.00mm, F.Cu at (96.4, 61.0)
- D1: footprint Connector_PinHeader_2.54mm:PinHeader_1x02_P2.54mm_Vertical -> LED_THT:LED_D5.0mm
- J3: value buck converter -> boost conv (OUT); footprint Connector_PinHeader_2.54mm:PinHeader_1x02_P2.54mm_Vertical -> TerminalBlock:TerminalBlock_Altech_AK300-2_P5.00mm
- J5: value BMI -> Light Sensor; footprint Connector_PinHeader_2.54mm:PinHeader_1x07_P2.54mm_Vertical -> Connector_PinHeader_2.54mm:PinHeader_1x04_P2.54mm_Vertical
- J6: value light sensor -> CAM UART; footprint Connector_PinHeader_2.54mm:PinHeader_1x05_P2.54mm_Vertical -> Connector_PinHeader_2.54mm:PinHeader_1x03_P2.54mm_Vertical
- J9: value battery + -> BMI; footprint Connector_PinHeader_2.54mm:PinHeader_1x01_P2.54mm_Vertical -> Connector_PinHeader_2.54mm:PinHeader_1x04_P2.54mm_Vertical
- Q1: footprint Package_TO_SOT_THT:TO-92_Inline -> Package_TO_SOT_THT:TO-92_Inline_Wide
- moved J9 66.7 mm to (165.0, 102.2), turned to 180 degrees
- moved J6 50.0 mm to (204.8, 126.8), turned to -90 degrees
- moved J3 31.6 mm to (152.8, 94.4), turned to -90 degrees
- moved C3 26.9 mm to (146.1, 105.2), turned to 0 degrees
- moved J5 23.0 mm to (184.0, 94.5), turned to 0 degrees
- moved D1 11.5 mm to (172.1, 119.4), turned to 180 degrees
- moved J7 10.2 mm to (99.5, 116.6), turned to 90 degrees
- moved Q1 3.57 mm to (155.9, 109.4)
- moved R3 3.00 mm to (195.8, 108.0)
- moved C2 2.64 mm to (113.4, 119.0), turned to 90 degrees
- moved J1 1.47 mm to (219.1, 55.4)
- moved J8 0.25 mm to (198.7, 50.0)
Connections:
- D1 pad 1: Net-(D1-K) -> GND
- J1 pad 3: Net-(D1-A) -> Net-(J1-Pin_3)
- J4 pad 3: Net-(D1-A) -> Net-(J1-Pin_3)
- J5 pad 1: unconnected-(J5-Pin_1-Pad1) -> Net-(J2-Pin_6)
- J5 pad 2: Net-(J2-Pin_3) -> Net-(J2-Pin_5)
- J5 pad 4: Net-(J2-Pin_5) -> Net-(J2-Pin_3)
- J6 pad 1: unconnected-(J6-Pin_1-Pad1) -> Net-(J6-Pin_1)
- J6 pad 2: Net-(J2-Pin_6) -> Net-(J6-Pin_2)
- J6 pad 3: Net-(J2-Pin_5) -> Net-(J6-Pin_3)
- J9 pad 1: Net-(J1-Pin_16) -> Net-(J2-Pin_3)
- R5 pad 1: GND -> Net-(D1-A)
- R5 pad 2: Net-(D1-K) -> Net-(J1-Pin_3)
- U2 pad GND1: unconnected-(U2-PadGND1) -> Net-(J6-Pin_3)
- U2 pad U0R: unconnected-(U2-PadU0R) -> Net-(J6-Pin_1)
- U2 pad U0T: unconnected-(U2-PadU0T) -> Net-(J6-Pin_2)
Routing:
- net GND: track 232.4 -> 384.1 mm
- net Net-(J2-Pin_9): track 288.1 -> 147.1 mm
- net Net-(J1-Pin_3): track 0.00 -> 121.5 mm
- net Net-(D1-A): track 113.6 -> 6.20 mm
- net VCC: track 145.7 -> 202.7 mm
- net Net-(J1-Pin_14): track 182.0 -> 165.2 mm
- net Net-(D1-K): track 11.8 -> 0.00 mm
- net Net-(J2-Pin_8): track 55.1 -> 64.7 mm
- net Net-(J2-Pin_7): track 45.9 -> 50.9 mm
- net Net-(J6-Pin_3): track 0.00 -> 4.41 mm
- net Net-(J6-Pin_2): track 0.00 -> 4.41 mm
- net Net-(J6-Pin_1): track 0.00 -> 4.41 mm
- net Net-(Q1-E): track 16.8 -> 13.0 mm
- net Net-(J2-Pin_4): track 55.5 -> 52.5 mm
- net Net-(J2-Pin_6): track 48.4 -> 45.4 mm
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Other:
- board size 135.3 x 80 mm -> 146.4 x 85.2 mm
