File: NEW.kicad_pcb (KiCad board)
At the start: 2 copper layers, 146.4 x 85.2 mm, 24 parts, among them J1 Screw_Terminal_01x16, J10 boost conv (IN), J11 Battery, J2 Screw_Terminal_01x16, J3 boost conv (OUT), J4 Infrared, J5 Light Sensor, J6 CAM UART, J7 servo, J8 Screw_Terminal_01x03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

Commit message: fixed proper wiring on power
Parts:
- removed U1: LM1117T-5.0, Package_TO_SOT_THT:TO-220-3_Horizontal_TabDown
- added Q2: IRLZ44N, Package_TO_SOT_THT:TO-220-3_Vertical, F.Cu at (139.5, 112.7)
- J8: value Screw_Terminal_01x03 -> LILYGO UART
- moved J8 45.6 mm to (219.1, 90.8), turned to -90 degrees
- moved C1 3.42 mm to (217.8, 104.6)
- moved J10 1.80 mm to (91.0, 101.0)
Connections:
- J1 pad 8: Net-(J1-Pin_8) -> unconnected-(J1-Pin_8-Pad8)
- J1 pad 9: Net-(J1-Pin_9) -> unconnected-(J1-Pin_9-Pad9)
- J2 pad 1: unconnected-(J2-Pin_1-Pad1) -> Net-(J2-Pin_1)
- J2 pad 2: unconnected-(J2-Pin_2-Pad2) -> Net-(J2-Pin_2)
- J8 pad 1: Net-(J1-Pin_9) -> Net-(J2-Pin_1)
- J8 pad 2: Net-(J1-Pin_8) -> Net-(J2-Pin_2)
- J8 pad 3: GND -> Net-(J2-Pin_4)
Routing:
- net GND: track 384.1 -> 439.7 mm
- net Net-(J2-Pin_7): track 50.9 -> 91.0 mm
- net Net-(J2-Pin_4): track 52.5 -> 82.7 mm
- net Net-(J2-Pin_9): track 147.1 -> 129.1 mm
- net Net-(J2-Pin_8): track 64.7 -> 77.0 mm
- net Net-(Q1-E): track 13.0 -> 24.6 mm
- net Net-(J1-Pin_9): track 5.42 -> 0.00 mm
- net Net-(J1-Pin_8): track 5.42 -> 0.00 mm
- net Net-(J2-Pin_1): track 0.00 -> 3.83 mm
- net Net-(J2-Pin_2): track 0.00 -> 3.83 mm
- net Net-(J1-Pin_14): track 165.2 -> 167.2 mm
- net Net-(J1-Pin_16): track 276.2 -> 277.4 mm
Other:
- board size 146.4 x 85.2 mm -> 148 x 85.2 mm
