File: rev3.kicad_pcb (KiCad board)
At the start: 2 copper layers, 148 x 100 mm, 25 parts, among them J1 Screw_Terminal_01x16, J10 boost conv (IN), J11 Battery, J2 Screw_Terminal_01x16, J3 boost conv (OUT), J4 Infrared, J5 Light Sensor, J6 CAM UART, J7 servo, J8 LILYGO UART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

Commit message: final rev
Parts:
- removed D2: 1N4007, Diode_THT:D_DO-41_SOD81_P12.70mm_Horizontal
- moved R1 19.1 mm to (201.2, 108.0), turned to 0 degrees
- moved Q2 18.6 mm to (139.5, 112.7), turned to -90 degrees
- moved J7 13.2 mm to (99.5, 116.6)
- moved Q1 12.0 mm to (155.9, 109.4)
- moved C2 11.7 mm to (113.4, 119.0)
- moved R2 10.8 mm to (223.0, 107.2)
- moved J6 10.8 mm to (204.8, 126.8)
- moved U2 10.8 mm to (193.5, 111.0)
- moved C1 10.8 mm to (217.8, 104.6)
- moved D1 10.0 mm to (172.1, 119.4)
- moved R4 10.0 mm to (156.0, 121.0)
- moved R5 10.0 mm to (164.0, 121.0)
- moved J4 9.89 mm to (178.0, 121.0)
- moved R3 2.53 mm to (195.8, 108.0), turned to 180 degrees
- moved J5 1.60 mm to (184.0, 94.5)
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Connections:
- C1 pad 2: Net-(Q2-D) -> GND
- Q2 pad 2: Net-(Q2-D) -> GND
- U2 pad GND2: Net-(Q2-D) -> GND
Routing:
- net Net-(Q2-D): track 93.7 -> 0.00 mm
- net GND: track 508.7 -> 439.7 mm
- net Net-(J2-Pin_9): track 66.3 -> 129.1 mm
- net VCC: track 237.5 -> 203.0 mm
- net Net-(J1-Pin_14): track 137.0 -> 167.2 mm
- net Net-(J2-Pin_8): track 48.4 -> 77.0 mm
- net Net-(J2-Pin_4): track 57.8 -> 82.7 mm
- net Net-(J1-Pin_3): track 137.8 -> 121.5 mm
- net Net-(J1-Pin_16): track 266.0 -> 277.4 mm
- net Net-(Q1-E): track 30.1 -> 24.6 mm
- net Net-(J2-Pin_7): track 95.5 -> 91.0 mm
- net Net-(J2-Pin_3): track 59.9 -> 55.8 mm
- net Net-(R1-Pad2): track 6.56 -> 8.92 mm
- net Net-(R2-Pad2): track 13.6 -> 15.6 mm
- net Net-(J2-Pin_5): track 50.1 -> 49.1 mm
Other:
- board size 148 x 100 mm -> 148 x 85.2 mm
